File: mfzh25_token/mfzh25_token.kicad_sch (KiCad schematic)
At the start: 36 parts, among them J2 Conn_02x03_Odd_Even

Commit message: almost there
Parts:
- TP1, TP2, TP3, TP4, TP5: footprint TestPoint:TestPoint_Pad_D4.0mm -> TestPoint:TestPoint_Pad_D1.5mm
- TP10: value TestPoint -> MF RR; footprint TestPoint:TestPoint_Pad_D2.0mm -> TestPoint:TestPoint_Pad_D1.5mm
- TP6: value TestPoint -> AA EI; footprint TestPoint:TestPoint_Pad_D2.0mm -> TestPoint:TestPoint_Pad_D1.5mm
- TP7: value TestPoint -> KR RF; footprint TestPoint:TestPoint_Pad_D2.0mm -> TestPoint:TestPoint_Pad_D1.5mm
- TP8: value TestPoint -> MI RE; footprint TestPoint:TestPoint_Pad_D2.0mm -> TestPoint:TestPoint_Pad_D1.5mm
- TP9: value TestPoint -> AR KF; footprint TestPoint:TestPoint_Pad_D2.0mm -> TestPoint:TestPoint_Pad_D1.5mm
Other:
- note added: "| M A K E R --|--------------- F | R G E N H --|--------------- A | L C B P X --|--------------- I | A Z U A Y --|--------------- R | R R C D O --|--------------- E | W R Q S R"
Changed lines of the file:
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@@
 		)
 	)
+	(text "  | M  A  K  E  R\n--|---------------\nF | R  G  E  N  H\n--|---------------\nA | L  C  B  P  X\n--|---------------\nI | A  Z  U  A  Y\n--|---------------\nR | R  R  C  D  O\n--|---------------\nE | W  R  Q  S  R"
+		(exclude_from_sim yes)
+		(at 172.974 80.518 0)
+		(effects
+			(font
+				(face "Adwaita Mono")
+				(size 1.27 1.27)
+				(thickness 0.1588)
+			)
+			(justify left)
+		)
+	)
 	(text "0805"
 		(exclude_from_sim no)
@@
 				)
 				(justify left)
+				(hide yes)
 			)
 		)
-		(property "Value" "TestPoint"
-			(at 139.7 76.7079 0)
+		(property "Value" "MI RE"
+			(at 139.7 75.4379 0)
 			(effects
 				(font
@@
 			)
 		)
-		(property "Footprint" "TestPoint:TestPoint_Pad_D2.0mm"
+		(property "Footprint" "TestPoint:TestPoint_Pad_D1.5mm"
 			(at 142.24 78.74 0)
 			(effects
@@
 			)
 		)
-		(property "Footprint" "TestPoint:TestPoint_Pad_D4.0mm"
+		(property "Footprint" "TestPoint:TestPoint_Pad_D1.5mm"
 			(at 88.9 104.14 0)
 			(effects
@@
 				)
 				(justify left)
+				(hide yes)
 			)
 		)
-		(property "Value" "TestPoint"
-			(at 139.7 51.3079 0)
+		(property "Value" "AA EI"
+			(at 139.7 50.0379 0)
 			(effects
 				(font
@@
 			)
 		)
-		(property "Footprint" "TestPoint:TestPoint_Pad_D2.0mm"
+		(property "Footprint" "TestPoint:TestPoint_Pad_D1.5mm"
 			(at 142.24 53.34 0)
 			(effects
@@
 				)
 				(justify left)
+				(hide yes)
 			)
 		)
-		(property "Value" "TestPoint"
-			(at 139.7 64.0079 0)
+		(property "Value" "KR RF"
+			(at 139.7 62.7379 0)
 			(effects
 				(font
@@
 			)
 		)
-		(property "Footprint" "TestPoint:TestPoint_Pad_D2.0mm"
+		(property "Footprint" "TestPoint:TestPoint_Pad_D1.5mm"
 			(at 142.24 66.04 0)
 			(effects
@@
 			)
 		)
-		(property "Footprint" "TestPoint:TestPoint_Pad_D4.0mm"
+		(property "Footprint" "TestPoint:TestPoint_Pad_D1.5mm"
 			(at 88.9 91.44 0)
 			(effects
@@
 			)
 		)
-		(property "Footprint" "TestPoint:TestPoint_Pad_D4.0mm"
+		(property "Footprint" "TestPoint:TestPoint_Pad_D1.5mm"
 			(at 88.9 53.34 0)
 			(effects
@@
 			)
 		)
-		(property "Footprint" "TestPoint:TestPoint_Pad_D4.0mm"
+		(property "Footprint" "TestPoint:TestPoint_Pad_D1.5mm"
 			(at 88.9 78.74 0)
 			(effects
@@
 				)
 				(justify left)
+				(hide yes)
 			)
 		)
-		(property "Value" "TestPoint"
-			(at 139.7 89.4079 0)
+		(property "Value" "AR KF"
+			(at 139.7 88.1379 0)
 			(effects
 				(font
@@
 			)
 		)
-		(property "Footprint" "TestPoint:TestPoint_Pad_D2.0mm"
+		(property "Footprint" "TestPoint:TestPoint_Pad_D1.5mm"
 			(at 142.24 91.44 0)
 			(effects
@@
 			)
 		)
-		(property "Footprint" "TestPoint:TestPoint_Pad_D4.0mm"
+		(property "Footprint" "TestPoint:TestPoint_Pad_D1.5mm"
 			(at 88.9 66.04 0)
 			(effects
@@
 				)
 				(justify left)
+				(hide yes)
 			)
 		)
-		(property "Value" "TestPoint"
-			(at 139.7 102.1079 0)
+		(property "Value" "MF RR"
+			(at 139.7 100.8379 0)
 			(effects
 				(font
@@
 			)
 		)
-		(property "Footprint" "TestPoint:TestPoint_Pad_D2.0mm"
+		(property "Footprint" "TestPoint:TestPoint_Pad_D1.5mm"
 			(at 142.24 104.14 0)
 			(effects
